Commit message: 9轴的urdf基本成熟了

File: 9_axis/urdf/9_axis.urdf (robot description, URDF)
Before this commit: robot 9_axis, 11 links, 10 joints
Links:
- link link04: mass 1.92823617150847 -> 15.1346479444998
- link link05: mass 5.84083453552761 -> 45.8465918633366
- link link06: mass 2.29995595587404 -> 18.0534564554839
- link link07: mass 0.705512031731609 -> 5.53782702890545
- link link08: mass 0.806930641656115 -> 6.33394466548073
- link link09: mass 0.180491791710468 -> 1.41689125820954
- link robobase: mass 0.01020659156849 -> 0.526598652051908
Joints:
- joint pris01: axis 0 0 0 -> 1 0 0; limit lower=0 upper=0 effort=0 velocity=0 -> lower=0 upper=20 effort=1000 velocity=1; origin xyz=2.4939 0.11 -14.901 rpy=1.5708 0 0 -> xyz=0 0 0 rpy=0 0 0
- joint pris02: axis 0 0 0 -> 0 1 0; limit lower=0 upper=0 effort=0 velocity=0 -> lower=-10 upper=2 effort=1000 velocity=1; origin xyz=0.6 18.841 -0.3 rpy=0 0 0 -> xyz=0 0 0 rpy=0 0 0
- joint pris03: axis 0 0 0 -> 0 0 1; limit lower=0 upper=0 effort=0 velocity=0 -> lower=0 upper=5 effort=1000 velocity=1; origin xyz=0 0 0.62434 rpy=0 0 0 -> xyz=0 0 0 rpy=0 0 0
- joint revo04: axis 0 0 0 -> 0 0 -1; limit lower=0 upper=0 effort=0 velocity=0 -> lower=-6.2832 upper=6.2832 effort=200 velocity=3.14; origin xyz=0 0.04 0 rpy=0 -1.4243 0 -> xyz=0 -0.00022535 0.12015 rpy=0 0 0
- joint revo05: axis 0 0 0 -> 0 0 1; limit lower=0 upper=0 effort=0 velocity=0 -> lower=-6.2832 upper=6.2832 effort=200 velocity=3.14; origin xyz=0.069608 -0.059809 0.066504 rpy=3.1416 -1.0811 1.5708 -> xyz=0 0 0 rpy=1.5708 0 0
- joint revo06: axis 0 0 0 -> 0 0 1; limit lower=0 upper=0 effort=0 velocity=0 -> lower=-6.2832 upper=6.2832 effort=200 velocity=3.14; origin xyz=0.789 0.0054421 0.22086 rpy=3.1416 0.1104 0 -> xyz=0.43 0 0 rpy=0 0 0
- joint revo07: axis 0 0 0 -> 0 0 -1; limit lower=-6.28 upper=6.28 effort=0 velocity=0 -> lower=-6.2832 upper=6.2832 effort=200 velocity=3.14; origin xyz=0.070737 -0.03895 0.053171 rpy=2.2874 0 -1.5708 -> xyz=0.3685 -1.185E-05 -0.114 rpy=0 0 0
- joint revo08: axis 0 0 0 -> 0 0 1; limit lower=6 upper=0 effort=0 velocity=0 -> lower=-6.2832 upper=6.2832 effort=200 velocity=3.14; origin xyz=0.0094486 -0.0455 -0.06734 rpy=1.4314 0 1.5708 -> xyz=0 -0.1135 0 rpy=1.5708 0 0
- joint revo09: axis 0 0 0 -> 0 0 1; limit lower=0 upper=0 effort=0 velocity=0 -> lower=-6.2832 upper=6.2832 effort=200 velocity=3.14; origin xyz=-0.041459 -0.039 -0.16284 rpy=3.1416 1.2693 3.1416 -> xyz=0 0.107 0 rpy=-1.5708 0 0
- joint robobase: origin xyz=-10.608 -7.5545 1.9876 rpy=-1.5708 0 0 -> xyz=-10.008 11.286 2.3119 rpy=-3.1415 0 0

Commit message: 加入了焊枪

File: 9_axis/urdf/9_axis.urdf (robot description, URDF)
Before this commit: robot 9_axis, 11 links, 10 joints
Links:
- added link weld_point, mass 0.012779; collision mesh filename=package://9_axis/meshes/weld_point.STL; visual mesh filename=package://9_axis/meshes/weld_point.STL
- added link welding_gun_base, mass 0.6969; collision mesh filename=package://9_axis/meshes/welding_gun_base.STL; visual mesh filename=package://9_axis/meshes/welding_gun_base.STL
- link base_link: mass 139.592927487695 -> 120.0
- link link_01: mass 6671.43699211194 -> 300.0
- link link_02: mass 40.148559695801 -> 40.0
- link link_03: mass 241.92854140384 -> 80.0
Joints:
- added joint fixed_point: type fixed, parent welding_gun_base, child weld_point, origin xyz=-0.248445440189498 0.01790694134073 0.117582478213501 rpy=-2.40735429840374 1.11493845934423 0.681057147859078
- added joint welding_gun_mount: type fixed, parent link09, child welding_gun_base, origin xyz=0 0 0 rpy=0 0 3.14
- joint pris03: limit lower=0 upper=5 effort=1000 velocity=1 -> lower=-1 upper=5 effort=1000 velocity=1
